File: ataro_v0.2/ataro_v0.2.kicad_pcb (KiCad board)
At the start: 4 copper layers, 202.6 x 151 mm, 85 parts, among them J1 4PIN, SW1 ESC, SW10 W, SW11 E, SW12 R, SW13 T, SW14 Y, SW15 CAPSLOCK, SW16 A, SW17 S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

Commit message: Final iteration of v0.2 for JLCPCB prod
Parts:
- removed G*** (x2): LOGO, LOGO
